File: Resistive-Soil-Humidity-Sensor/Resistive-Soil-Humidity-Sensor.sch (KiCad schematic (older format))
At the start: 8 parts, among them Q1 BC547

Commit message: add pcb-layout
Parts:
- removed Probe1: Jumper, symbol Device:Jumper
- added H1, H2: MountingHole_Pad, custom_libraryies:MountingHole.1.8mm, symbol Mechanical:MountingHole_Pad
Connections:
- net at Q1.2 (B), RV1.2: now also H1.1
- net at BZ1.1 (-), R1.1, Voltage-Reg1.3 (OUT): now also H2.1
Changed lines of the file:
@@
-	1    0    0    -1
-$EndComp
-$Comp
-L Device:Jumper Probe1
-U 1 1 6378CB33
-P 8800 5000
-F 0 "Probe1" H 8800 5264 50  0000 C CNN
-F 1 "Jumper" H 8800 5173 50  0000 C CNN
-F 2 "" H 8800 5000 50  0001 C CNN
-F 3 "~" H 8800 5000 50  0001 C CNN
-	1    8800 5000
 	1    0    0    -1
 $EndComp
@@
 	9600 5350 9600 5000
 Wire Wire Line
-	9100 5000 9600 5000
-Wire Wire Line
 	9600 5350 9600 5900
 Wire Wire Line
 	9500 5900 9600 5900
 Connection ~ 9600 5350
+Wire Wire Line
+	8500 5000 8650 5000
+Wire Wire Line
+	9000 5000 9600 5000
+$Comp
+L Mechanical:MountingHole_Pad H2
+U 1 1 63810D2C
+P 8650 4900
+F 0 "H2" H 8750 4905 50  0000 L CNN
+F 1 "MountingHole_Pad" H 8750 4860 50  0001 L CNN
+F 2 "custom_libraryies:MountingHole.1.8mm" H 8650 4900 50  0001 C CNN
+F 3 "~" H 8650 4900 50  0001 C CNN
+	1    8650 4900
+	1    0    0    -1
+$EndComp
+$Comp
+L Mechanical:MountingHole_Pad H1
+U 1 1 63810E2E
+P 9000 4900
+F 0 "H1" H 9100 4905 50  0000 L CNN
+F 1 "MountingHole_Pad" H 9100 4860 50  0001 L CNN
+F 2 "custom_libraryies:MountingHole.1.8mm" H 9000 4900 50  0001 C CNN
+F 3 "~" H 9000 4900 50  0001 C CNN
+	1    9000 4900
+	1    0    0    -1
+$EndComp
 $EndSCHEMATC

Commit message: pull from repo
Parts:
- BZ1: footprint (none) -> Buzzer_Beeper:Buzzer_12x9.5RM7.6
Changed lines of the file:
@@
 F 0 "BZ1" H 10553 5029 50  0000 L CNN
 F 1 "Buzzer" H 10553 4938 50  0000 L CNN
-F 2 "" V 10375 5100 50  0001 C CNN
+F 2 "Buzzer_Beeper:Buzzer_12x9.5RM7.6" V 10375 5100 50  0001 C CNN
 F 3 "~" V 10375 5100 50  0001 C CNN
 	1    10400 5000
