File: Resistive-Soil-Humidity-Sensor/Resistive-Soil-Humidity-Sensor.kicad_sch (KiCad schematic)
At the start: 9 parts, among them Q1 BC547, U1 L7805CV

Commit message: update the design for new power supply
Parts:
- H1, H2: footprint custom_libraryies:MountingHole.1.8mm -> Connector_Pin:Pin_D0.9mm_L10.0mm_W2.4mm_FlatFork
Changed lines of the file:
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@@
       (effects (font (size 1.27 1.27)) (justify left) hide)
     )
-    (property "Footprint" "custom_libraryies:MountingHole.1.8mm" (id 2) (at 219.71 124.46 0)
+    (property "Footprint" "Connector_Pin:Pin_D0.9mm_L10.0mm_W2.4mm_FlatFork" (id 2) (at 219.71 124.46 0)
       (effects (font (size 1.27 1.27)) hide)
     )
@@
       (effects (font (size 1.27 1.27)) (justify left) hide)
     )
-    (property "Footprint" "custom_libraryies:MountingHole.1.8mm" (id 2) (at 228.6 124.46 0)
+    (property "Footprint" "Connector_Pin:Pin_D0.9mm_L10.0mm_W2.4mm_FlatFork" (id 2) (at 228.6 124.46 0)
       (effects (font (size 1.27 1.27)) hide)
     )
@@
       (reference "D1") (unit 1) (value "LED") (footprint "LED_THT:LED_D3.0mm_FlatTop")
     )
-    (path "/00000000-0000-0000-0000-000063810e2e"
-      (reference "H1") (unit 1) (value "MountingHole_Pad") (footprint "custom_libraryies:MountingHole.1.8mm")
+    (path "/053aa4e3-3c22-47af-931c-1d193f4e41c2"
+      (reference "H1") (unit 1) (value "MountingHole_Pad") (footprint "Connector_Pin:Pin_D0.9mm_L10.0mm_W2.4mm_FlatFork")
     )
     (path "/00000000-0000-0000-0000-000063810d2c"
-      (reference "H2") (unit 1) (value "MountingHole_Pad") (footprint "custom_libraryies:MountingHole.1.8mm")
+      (reference "H2") (unit 1) (value "MountingHole_Pad") (footprint "Connector_Pin:Pin_D0.9mm_L10.0mm_W2.4mm_FlatFork")
     )
     (path "/00000000-0000-0000-0000-00006378b088"

Commit message: add new pcb layout pdf's
Parts:
- Q1: footprint Package_TO_SOT_THT:TO-92_Inline -> Package_TO_SOT_THT:TO-92_Inline2-bigger
Changed lines of the file:
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@@
       (effects (font (size 1.27 1.27)) (justify left))
     )
-    (property "Footprint" "Package_TO_SOT_THT:TO-92_Inline" (id 2) (at 254 137.795 0)
+    (property "Footprint" "Package_TO_SOT_THT:TO-92_Inline2-bigger" (id 2) (at 254 137.795 0)
       (effects (font (size 1.27 1.27) italic) (justify left) hide)
     )
@@
     )
     (path "/00000000-0000-0000-0000-00006378b088"
-      (reference "Q1") (unit 1) (value "BC547") (footprint "Package_TO_SOT_THT:TO-92_Inline")
+      (reference "Q1") (unit 1) (value "BC547") (footprint "Package_TO_SOT_THT:TO-92_Inline2-bigger")
     )
     (path "/00000000-0000-0000-0000-00006378be2c"
