File: Resistive-Soil-Humidity-Sensor/beforeexport.kicad_pcb (KiCad board)
At the start: 2 copper layers, 40 parts, among them Q1 BC547, U1 L7805CV

Commit message: add new pcb layout pdf's
Parts:
- removed the 9V1 at (141.4, 34.2)
- removed the 9V1 at (165.7, 117.5)
- removed the 9V1 at (51.5, 117.8)
- removed the 9V1 at (53.2, 35.6)
- removed the D1 at (40.0, 23.8)
- removed the D1 at (152.5, 105.7)
- removed the D1 at (128.2, 22.4)
- removed the D1 at (38.3, 106.0)
- removed the H1 at (188.2, 105.7)
- removed the H1 at (73.9, 106.0)
- removed the H1 at (75.6, 23.8)
- removed the H1 at (163.8, 22.4)
- removed the H2 at (188.2, 108.5)
- removed the H2 at (75.6, 26.6)
- removed the H2 at (163.8, 25.2)
- removed the H2 at (73.9, 108.8)
- removed the Q1 at (57.2, 23.8)
- removed the Q1 at (55.5, 106.0)
- removed the Q1 at (169.7, 105.7)
- removed the Q1 at (145.3, 22.4)
- removed the Q1 at (242.5, 22.8)
- removed the R1 at (126.1, 26.7)
- removed the R1 at (38.0, 28.1)
- removed the R1 at (150.5, 110.0)
- removed the R1 at (36.3, 110.3)
- removed the RV1 at (167.2, 129.7)
- removed the RV1 at (53.0, 129.9)
- removed the RV1 at (142.9, 46.3)
- removed the RV1 at (54.7, 47.8)
- removed the U1 at (36.9, 121.0)
- removed the U1 at (151.1, 120.7)
- removed the U1 at (126.7, 37.4)
- removed the U1 at (38.6, 38.8)
- added 9V1: BH9VPC, BHVPC-BatteryHolder:BAT_BH9VPC, B.Cu at (145.7, 33.9)
- added 9V1: BH9VPC, BHVPC-BatteryHolder:BAT_BH9VPC, B.Cu at (50.8, 98.1)
- added 9V1: BH9VPC, BHVPC-BatteryHolder:BAT_BH9VPC, B.Cu at (141.6, 96.6)
- added 9V1: BH9VPC, BHVPC-BatteryHolder:BAT_BH9VPC, B.Cu at (234.4, 97.3)
- added 9V1: BH9VPC, BHVPC-BatteryHolder:BAT_BH9VPC, B.Cu at (54.9, 35.4)
- added D1: LED, LED_THT:LED_D3.0mm_FlatTop, F.Cu at (132.5, 22.1)
- added D1: LED, LED_THT:LED_D3.0mm_FlatTop, F.Cu at (128.4, 84.8)
- added D1: LED, LED_THT:LED_D3.0mm_FlatTop, F.Cu at (221.2, 85.4)
- added D1: LED, LED_THT:LED_D3.0mm_FlatTop, F.Cu at (37.6, 86.3)
- added D1: LED, LED_THT:LED_D3.0mm_FlatTop, F.Cu at (41.7, 23.6)
- added H1: MountingHole_Pad, Connector_Pin:Pin_D0.9mm_L10.0mm_W2.4mm_FlatFork, F.Cu at (256.8, 85.4)
- added H1: MountingHole_Pad, Connector_Pin:Pin_D0.9mm_L10.0mm_W2.4mm_FlatFork, F.Cu at (73.2, 86.3)
- added H1: MountingHole_Pad, Connector_Pin:Pin_D0.9mm_L10.0mm_W2.4mm_FlatFork, F.Cu at (164.0, 84.8)
- added H1: MountingHole_Pad, Connector_Pin:Pin_D0.9mm_L10.0mm_W2.4mm_FlatFork, F.Cu at (168.1, 22.1)
- added H1: MountingHole_Pad, Connector_Pin:Pin_D0.9mm_L10.0mm_W2.4mm_FlatFork, F.Cu at (77.3, 23.6)
- added H2: MountingHole_Pad, Connector_Pin:Pin_D0.9mm_L10.0mm_W2.4mm_FlatFork, F.Cu at (168.1, 24.9)
- added H2: MountingHole_Pad, Connector_Pin:Pin_D0.9mm_L10.0mm_W2.4mm_FlatFork, F.Cu at (77.3, 26.4)
- added H2: MountingHole_Pad, Connector_Pin:Pin_D0.9mm_L10.0mm_W2.4mm_FlatFork, F.Cu at (73.2, 89.1)
- added H2: MountingHole_Pad, Connector_Pin:Pin_D0.9mm_L10.0mm_W2.4mm_FlatFork, F.Cu at (256.8, 88.3)
- added H2: MountingHole_Pad, Connector_Pin:Pin_D0.9mm_L10.0mm_W2.4mm_FlatFork, F.Cu at (164.0, 87.6)
- added Q1: BC547, Package_TO_SOT_THT:TO-92_Inline2-bigger, B.Cu at (53.8, 86.6)
- added Q1: BC547, Package_TO_SOT_THT:TO-92_Inline2-bigger, B.Cu at (144.5, 85.1)
- added Q1: BC547, Package_TO_SOT_THT:TO-92_Inline2-bigger, B.Cu at (241.5, 23.0)
- added Q1: BC547, Package_TO_SOT_THT:TO-92_Inline2-bigger, B.Cu at (237.4, 85.7)
- added Q1: BC547, Package_TO_SOT_THT:TO-92_Inline2-bigger, B.Cu at (57.9, 23.9)
- added Q1: BC547, Package_TO_SOT_THT:TO-92_Inline2-bigger, B.Cu at (148.6, 22.3)
- added R1: 1kohm, Resistor_SMD:R_0402_1005Metric, B.Cu at (39.7, 27.9)
- added R1: 1kohm, Resistor_SMD:R_0402_1005Metric, B.Cu at (126.3, 89.1)
- added R1: 1kohm, Resistor_SMD:R_0402_1005Metric, B.Cu at (130.5, 26.4)
- added R1: 1kohm, Resistor_SMD:R_0402_1005Metric, B.Cu at (35.6, 90.6)
- added R1: 1kohm, Resistor_SMD:R_0402_1005Metric, B.Cu at (219.2, 89.8)
- added RV1: R_POT, Potentiometer_THT:Potentiometer_Bourns_3266Y_Vertical, F.Cu at (143.1, 108.8)
- added RV1: R_POT, Potentiometer_THT:Potentiometer_Bourns_3266Y_Vertical, F.Cu at (52.3, 110.3)
- added RV1: R_POT, Potentiometer_THT:Potentiometer_Bourns_3266Y_Vertical, F.Cu at (235.9, 109.4)
- added RV1: R_POT, Potentiometer_THT:Potentiometer_Bourns_3266Y_Vertical, F.Cu at (147.2, 46.0)
- added RV1: R_POT, Potentiometer_THT:Potentiometer_Bourns_3266Y_Vertical, F.Cu at (56.4, 47.6)
- added U1: L7805CV, L7805CV-Vreg:TO255P1040X460X1968-3, F.Cu at (126.9, 99.8)
- added U1: L7805CV, L7805CV-Vreg:TO255P1040X460X1968-3, F.Cu at (219.8, 100.4)
- added U1: L7805CV, L7805CV-Vreg:TO255P1040X460X1968-3, F.Cu at (36.1, 101.3)
- added U1: L7805CV, L7805CV-Vreg:TO255P1040X460X1968-3, F.Cu at (40.3, 38.6)
- added U1: L7805CV, L7805CV-Vreg:TO255P1040X460X1968-3, F.Cu at (131.0, 37.1)
Routing:
- net Net-(9V1-Pad-): track 315.7 -> 382.8 mm
- net Net-(H1-Pad1): track 222.5 -> 272.3 mm
- net Net-(BZ1-Pad1): track 216.9 -> 260.3 mm
- net Net-(BZ1-Pad2): track 86.0 -> 99.1 mm
- net Net-(9V1-Pad+): track 58.1 -> 69.7 mm
- net Net-(D1-Pad2): track 21.8 -> 26.1 mm

Commit message: added buzzer
Parts:
- removed the 9V1 at (145.7, 33.9)
- removed the 9V1 at (50.8, 98.1)
- removed the 9V1 at (141.6, 96.6)
- removed the 9V1 at (234.4, 97.3)
- removed the 9V1 at (54.9, 35.4)
- removed the D1 at (132.5, 22.1)
- removed the D1 at (128.4, 84.8)
- removed the D1 at (221.2, 85.4)
- removed the D1 at (37.6, 86.3)
- removed the D1 at (41.7, 23.6)
- removed the H1 at (256.8, 85.4)
- removed the H1 at (73.2, 86.3)
- removed the H1 at (164.0, 84.8)
- removed the H1 at (168.1, 22.1)
- removed the H1 at (77.3, 23.6)
- removed the H2 at (168.1, 24.9)
- removed the H2 at (77.3, 26.4)
- removed the H2 at (73.2, 89.1)
- removed the H2 at (256.8, 88.3)
- removed the H2 at (164.0, 87.6)
- removed the Q1 at (53.8, 86.6)
- removed the Q1 at (144.5, 85.1)
- removed the Q1 at (237.4, 85.7)
- removed the Q1 at (57.9, 23.9)
- removed the Q1 at (148.6, 22.3)
- removed the R1 at (39.7, 27.9)
- removed the R1 at (126.3, 89.1)
- removed the R1 at (130.5, 26.4)
- removed the R1 at (35.6, 90.6)
- removed the R1 at (219.2, 89.8)
- removed the RV1 at (143.1, 108.8)
- removed the RV1 at (52.3, 110.3)
- removed the RV1 at (235.9, 109.4)
- removed the RV1 at (147.2, 46.0)
- removed the RV1 at (56.4, 47.6)
- removed the U1 at (126.9, 99.8)
- removed the U1 at (219.8, 100.4)
- removed the U1 at (36.1, 101.3)
- removed the U1 at (40.3, 38.6)
- removed the U1 at (131.0, 37.1)
- added 9V1: BH9VPC, BHVPC-BatteryHolder:BAT_BH9VPC, B.Cu at (141.3, 90.8)
- added 9V1: BH9VPC, BHVPC-BatteryHolder:BAT_BH9VPC, B.Cu at (48.5, 33.4)
- added 9V1: BH9VPC, BHVPC-BatteryHolder:BAT_BH9VPC, B.Cu at (237.2, 90.7)
- added 9V1: BH9VPC, BHVPC-BatteryHolder:BAT_BH9VPC, B.Cu at (47.1, 89.5)
- added 9V1: BH9VPC, BHVPC-BatteryHolder:BAT_BH9VPC, B.Cu at (142.3, 34.6)
- added BZ1: Buzzer, Buzzer_Beeper:Buzzer_12x9.5RM7.6, F.Cu at (135.6, 46.7)
- added BZ1: Buzzer, Buzzer_Beeper:Buzzer_12x9.5RM7.6, F.Cu at (134.6, 103.0)
- added D1: LED, LED_THT:LED_D3.0mm_FlatTop, F.Cu at (33.9, 77.7)
- added D1: LED, LED_THT:LED_D3.0mm_FlatTop, F.Cu at (128.1, 79.0)
- added D1: LED, LED_THT:LED_D3.0mm_FlatTop, F.Cu at (224.0, 78.8)
- added D1: LED, LED_THT:LED_D3.0mm_FlatTop, F.Cu at (35.3, 21.6)
- added D1: LED, LED_THT:LED_D3.0mm_FlatTop, F.Cu at (129.1, 22.7)
- added H1: MountingHole_Pad, Connector_Pin:Pin_D0.9mm_L10.0mm_W2.4mm_FlatFork, F.Cu at (70.9, 21.6)
- added H1: MountingHole_Pad, Connector_Pin:Pin_D0.9mm_L10.0mm_W2.4mm_FlatFork, F.Cu at (69.6, 77.7)
- added H1: MountingHole_Pad, Connector_Pin:Pin_D0.9mm_L10.0mm_W2.4mm_FlatFork, F.Cu at (163.8, 79.0)
- added H1: MountingHole_Pad, Connector_Pin:Pin_D0.9mm_L10.0mm_W2.4mm_FlatFork, F.Cu at (164.7, 22.7)
- added H1: MountingHole_Pad, Connector_Pin:Pin_D0.9mm_L10.0mm_W2.4mm_FlatFork, F.Cu at (259.6, 78.8)
- added H2: MountingHole_Pad, Connector_Pin:Pin_D0.9mm_L10.0mm_W2.4mm_FlatFork, F.Cu at (163.8, 81.8)
- added H2: MountingHole_Pad, Connector_Pin:Pin_D0.9mm_L10.0mm_W2.4mm_FlatFork, F.Cu at (259.6, 81.7)
- added H2: MountingHole_Pad, Connector_Pin:Pin_D0.9mm_L10.0mm_W2.4mm_FlatFork, F.Cu at (69.6, 80.5)
- added H2: MountingHole_Pad, Connector_Pin:Pin_D0.9mm_L10.0mm_W2.4mm_FlatFork, F.Cu at (70.9, 24.4)
- added H2: MountingHole_Pad, Connector_Pin:Pin_D0.9mm_L10.0mm_W2.4mm_FlatFork, F.Cu at (164.7, 25.6)
- added Q1: BC547, Package_TO_SOT_THT:TO-92_Inline2-bigger, B.Cu at (51.5, 21.8)
- added Q1: BC547, Package_TO_SOT_THT:TO-92_Inline2-bigger, B.Cu at (240.1, 79.1)
- added Q1: BC547, Package_TO_SOT_THT:TO-92_Inline2-bigger, B.Cu at (50.1, 78.0)
- added Q1: BC547, Package_TO_SOT_THT:TO-92_Inline2-bigger, B.Cu at (144.3, 79.3)
- added Q1: BC547, Package_TO_SOT_THT:TO-92_Inline2-bigger, B.Cu at (145.3, 23.0)
- added R1: 1kohm, Resistor_SMD:R_0402_1005Metric, B.Cu at (31.9, 82.0)
- added R1: 1kohm, Resistor_SMD:R_0402_1005Metric, B.Cu at (33.3, 25.9)
- added R1: 1kohm, Resistor_SMD:R_0402_1005Metric, B.Cu at (126.1, 83.3)
- added R1: 1kohm, Resistor_SMD:R_0402_1005Metric, B.Cu at (127.1, 27.1)
- added R1: 1kohm, Resistor_SMD:R_0402_1005Metric, B.Cu at (222.0, 83.2)
- added RV1: R_POT, Potentiometer_THT:editted_Potentiometer_Bourns_3266Y_Vertical, F.Cu at (143.1, 46.9)
- added RV1: R_POT, Potentiometer_THT:editted_Potentiometer_Bourns_3266Y_Vertical, F.Cu at (49.3, 45.8)
- added RV1: R_POT, Potentiometer_THT:editted_Potentiometer_Bourns_3266Y_Vertical, F.Cu at (47.9, 101.9)
- added RV1: R_POT, Potentiometer_THT:editted_Potentiometer_Bourns_3266Y_Vertical, F.Cu at (238.0, 103.0)
- added RV1: R_POT, Potentiometer_THT:editted_Potentiometer_Bourns_3266Y_Vertical, F.Cu at (142.1, 103.2)
- added U1: L7805CV, L7805CV-Vreg:TO255P1040X460X1968-3, F.Cu at (126.7, 94.0)
- added U1: L7805CV, L7805CV-Vreg:TO255P1040X460X1968-3, F.Cu at (33.8, 36.6)
- added U1: L7805CV, L7805CV-Vreg:TO255P1040X460X1968-3, F.Cu at (222.5, 93.8)
- added U1: L7805CV, L7805CV-Vreg:TO255P1040X460X1968-3, F.Cu at (127.7, 37.7)
- added U1: L7805CV, L7805CV-Vreg:TO255P1040X460X1968-3, F.Cu at (32.5, 92.7)
- RV1: footprint Potentiometer_THT:Potentiometer_Bourns_3266Y_Vertical -> Potentiometer_THT:editted_Potentiometer_Bourns_3266Y_Vertical
- moved RV1 0.76 mm to (239.3, 46.9)
Routing:
- net Net-(BZ1-Pad2): track 99.1 -> 139.3 mm
- net Net-(BZ1-Pad1): track 260.3 -> 295.1 mm
- net Net-(9V1-Pad-): track 382.8 -> 402.4 mm
- net Net-(H1-Pad1): track 272.3 -> 282.2 mm
