File: Esp-Based-Soil-Humidity-Monitoring-Device-R/Esp-Based-Soil-Humidity-Monitoring-Device-R.sch (KiCad schematic (older format))
At the start: 31 parts, among them IC1 ESP-12F, IC2 CP2102-GMR_NRND, J1 629105136821, Q1 Q_DUAL_NPN_NPN_E1B1C2E2B2C1, SW1 SW_DIP_x01, SW2 SW_DIP_x01

Commit message: finish USB Section
Parts:
- removed D? (x4): DIODE_SCHOTTKY, symbol freetronics_schematic:DIODE_SCHOTTKY
- added D1: LED, symbol Device:LED
- added R7: 680R, symbol Device:R
- added U?: SRV05-4, Package_TO_SOT_SMD:SOT-23-6, symbol Power_Protection:SRV05-4
Connections:
- wire segments 109 -> 118
Changed lines of the file:
@@
 $EndComp
 $Comp
-L freetronics_schematic:DIODE_SCHOTTKY D?
-U 1 1 638DFC4C
-P 2100 4050
-F 0 "D?" V 1750 4050 40  0000 R CNN
-F 1 "DIODE_SCHOTTKY" V 1800 4250 40  0001 R CNN
-F 2 "" H 2100 4050 60  0000 C CNN
-F 3 "" H 2100 4050 60  0000 C CNN
-	1    2100 4050
+L Power_Protection:SRV05-4 U?
+U 1 1 638F3A01
+P 2100 4900
+F 0 "U?" H 2500 4550 50  0000 C CNN
+F 1 "SRV05-4" H 2350 4450 50  0000 C CNN
+F 2 "Package_TO_SOT_SMD:SOT-23-6" H 2800 4450 50  0001 C CNN
+F 3 "http://www.onsemi.com/pub/Collateral/SRV05-4-D.PDF" H 2100 4900 50  0001 C CNN
+	1    2100 4900
+	1    0    0    -1
+$EndComp
+Wire Wire Line
+	1200 4350 2100 4350
+Wire Wire Line
+	2100 4350 2100 4400
+Wire Wire Line
+	1200 4250 1600 4250
+Wire Wire Line
+	1600 4250 1600 4800
+Wire Wire Line
+	1600 5000 1450 5000
+Wire Wire Line
+	1450 5000 1450 4150
+Wire Wire Line
+	1450 4150 1200 4150
+$Comp
+L power:GND #PWR?
+U 1 1 63904A57
+P 1300 3950
+F 0 "#PWR?" H 1300 3700 50  0001 C CNN
+F 1 "GND" V 1305 3822 50  0000 R CNN
+F 2 "" H 1300 3950 50  0001 C CNN
+F 3 "" H 1300 3950 50  0001 C CNN
+	1    1300 3950
 	0    -1   -1   0
 $EndComp
 $Comp
-L freetronics_schematic:DIODE_SCHOTTKY D?
-U 1 1 638E2608
-P 1950 4050
-F 0 "D?" V 1600 4050 40  0000 R CNN
-F 1 "DIODE_SCHOTTKY" V 1650 4250 40  0001 R CNN
-F 2 "" H 1950 4050 60  0000 C CNN
-F 3 "" H 1950 4050 60  0000 C CNN
-	1    1950 4050
-	0    -1   -1   0
+L power:GND #PWR?
+U 1 1 63904B80
+P 2100 5500
+F 0 "#PWR?" H 2100 5250 50  0001 C CNN
+F 1 "GND" V 2105 5372 50  0000 R CNN
+F 2 "" H 2100 5500 50  0001 C CNN
+F 3 "" H 2100 5500 50  0001 C CNN
+	1    2100 5500
+	1    0    0    -1
+$EndComp
+Wire Wire Line
+	1300 3950 1200 3950
+Wire Wire Line
+	2100 5400 2100 5500
+Wire Wire Line
+	1600 4250 2600 4250
+Connection ~ 1600 4250
+Wire Wire Line
+	1450 4150 2600 4150
+Connection ~ 1450 4150
+Text Label 2600 4150 2    39   Italic 0
+USB_DP
+Text Label 2600 4250 2    39   Italic 0
+USB_DN
+$Comp
+L power:GND #PWR?
+U 1 1 63915497
+P 2750 4400
+F 0 "#PWR?" H 2750 4150 50  0001 C CNN
+F 1 "GND" V 2755 4272 50  0000 R CNN
+F 2 "" H 2750 4400 50  0001 C CNN
+F 3 "" H 2750 4400 50  0001 C CNN
+	1    2750 4400
+	0    1    1    0
 $EndComp
 $Comp
-L freetronics_schematic:DIODE_SCHOTTKY D?
-U 1 1 638E2664
-P 2250 4050
-F 0 "D?" V 1900 4050 40  0000 R CNN
-F 1 "DIODE_SCHOTTKY" V 1950 4250 40  0001 R CNN
-F 2 "" H 2250 4050 60  0000 C CNN
-F 3 "" H 2250 4050 60  0000 C CNN
-	1    2250 4050
-	0    -1   -1   0
+L Device:R R7
+U 1 1 63918CD6
+P 3400 4400
+F 0 "R7" V 3500 4400 50  0000 C CNN
+F 1 "680R" V 3400 4400 39  0000 C CNN
+F 2 "" V 3330 4400 50  0001 C CNN
+F 3 "~" H 3400 4400 50  0001 C CNN
+	1    3400 4400
+	0    1    1    0
 $EndComp
 $Comp
-L freetronics_schematic:DIODE_SCHOTTKY D?
-U 1 1 638E26D0
-P 2400 4050
-F 0 "D?" V 2050 4050 40  0000 R CNN
-F 1 "DIODE_SCHOTTKY" V 2100 4250 40  0001 R CNN
-F 2 "" H 2400 4050 60  0000 C CNN
-F 3 "" H 2400 4050 60  0000 C CNN
-	1    2400 4050
-	0    -1   -1   0
+L Device:LED D1
+U 1 1 63919092
+P 3000 4400
+F 0 "D1" H 2991 4616 50  0000 C CNN
+F 1 "LED" H 2991 4525 50  0000 C CNN
+F 2 "" H 3000 4400 50  0001 C CNN
+F 3 "~" H 3000 4400 50  0001 C CNN
+	1    3000 4400
+	1    0    0    -1
 $EndComp
 Wire Wire Line
-	1950 4250 2100 4250
-Connection ~ 2100 4250
+	2750 4400 2850 4400
 Wire Wire Line
-	2100 4250 2200 4250
-Connection ~ 2250 4250
+	3150 4400 3250 4400
 Wire Wire Line
-	2250 4250 2400 4250
-Wire Wire Line
-	2200 4250 2200 4500
-Connection ~ 2200 4250
-Wire Wire Line
-	2200 4250 2250 4250
-$Comp
-L power:GND #PWR?
-U 1 1 638E8115
-P 2200 4500
-F 0 "#PWR?" H 2200 4250 50  0001 C CNN
-F 1 "GND" V 2205 4372 50  0000 R CNN
-F 2 "" H 2200 4500 50  0001 C CNN
-F 3 "" H 2200 4500 50  0001 C CNN
-	1    2200 4500
-	1    0    0    -1
-$EndComp
+	3550 4400 3650 4400
+Text GLabel 3650 4400 2    39   Input Italic 0
+VBUS
 $EndSCHEMATC

Commit message: finish Battery management
Parts:
- added C3: 2.2uF/6.3V, symbol Device:C_Small
- added D?: LED, symbol Device:LED
- added R? (x2): 680R, symbol Device:R
- added U?: LTC4054ES5-4.2, Package_TO_SOT_SMD:TSOT-23-5, symbol Battery_Management:LTC4054ES5-4.2
Connections:
- net labels added: CHARGER
- wire segments 118 -> 133
Other:
- note added: "Battery Management/Charger Section\n\n"
- note added: "USB to UART Section"
- note removed: "USB to UART"

Commit message: finish Reverse Polarity Protection
Parts:
- added BT1: Battery_Cell, symbol Device:Battery_Cell
- added C6: 470pF/10V, symbol Device:C_Small
- added C7: 10uF/6.3V, symbol Device:C_Small
- added C8: 0.1uF/6.3V, symbol Device:C_Small
- added D2: SS14, digikey-footprints:DO-214AC, symbol dk_Diodes-Rectifiers-Single:SS14
- added IC3: MIC5219-3_3YM5-TR, digikey-footprints:SOT-753, symbol dk_PMIC-Voltage-Regulators-Linear:MIC5219-3_3YM5-TR
- added Q2: SI2301, SI2305TP, symbol SI2301:SI2301
- added R14: 100k, symbol Device:R
- gave numbers to parts that had none: 7
- renumbered deep-sleep-jumper to deep-sleep-jumper1
Connections:
- net labels added: 3.3V-Reg
- wire segments 133 -> 163
Other:
- note added: "Charging Section\n"
- note added: "Reverse Polarity Protection\n\n"
- note added: "USB Section"
- note removed: "Battery Management/Charger Section\n\n"
